File: Mini12.sch (EAGLE design)
At the start: 61 parts, among them IC1 LM833N, IC2 LM339N, Q1 2N3904

Commit message: Finished schematic
Parts:
- removed C2, C3: 47uF, rcl:CPOL-EUE2.5-6
- removed C7: 1000uF, rcl:CPOL-EUE5-10.5
- removed Q1: 2N3904, transistor-npn:2N3904
- removed R1: 560Ω, rcl:R-EU_0207/10
- removed R2: 100Ω, rcl:R-EU_0207/10
- removed R5, R6: 1kΩ, rcl:R-EU_0207/10
- removed VR1: 10kΩ, bourns:3362U
- removed VR2: 100kΩ, bourns:3362U
- added Q2, Q5: 2N3904, transistor-npn:2N3904
- added Q3, Q6: 2N3906, transistor-pnp:2N3906
- added Q4, Q7: TIP31C, transistor-npn:TIP31C
- added T1, T2: TIP32C, transistor:TIP32C
Connections:
- removed net INPUT: C2.+, R5.2, R6.2
- removed net N$1: C7.-, VR2.2
- removed net N$4: D1.A, D2.C, R_OUT.1
- removed net N$42: C3.+, Q1.E, R2.2
- removed net N$47: C2.-, Q1.B, VR1.2
- removed net N$8: D3.A, D4.C, L_OUT.1
- removed net PREOUTPUT: C7.+, Q1.C, R1.1
- removed net VCC: R1.2, VR1.3, VR2.3
- new net N$24: Q2.E, Q4.B
- new net N$25: Q3.E, T1.B
- new net N$26: D1.A, D2.C, Q4.E, R7.2, R_OUT.1, T1.E
- new net N$27: IC1A.OUT, Q2.B, Q3.B
- new net N$31: Q5.E, Q7.B
- new net N$32: Q6.E, T2.B
- new net N$33: D3.A, D4.C, L_OUT.1, Q7.E, R11.2, T2.E
- new net N$34: IC1B.OUT, Q5.B, Q6.B
- net GND: no longer C3.-, R2.1, VR1.1, VR2.1
- net V+: now also Q2.C, Q4.C, Q5.C, Q7.C
- net V-: now also Q3.C, Q6.C, T1.C, T2.C
Other:
- note removed: "Amplifier"
- note removed: "Power Amplifier"
- moved on the sheet: AUDIO_IN1, AUDIO_IN2, AUDIO_IN3, C6, D1, D2, D3, D4, IC1B, L_OUT, R10, R11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
